File: Pi_Zero_RS232_DB25_Hat.kicad_pcb (KiCad board)
At the start: 2 copper layers, 65.2 x 42 mm, 10 parts, among them J1 Raspberry_Pi_2_3, J2 DB25_Female_MountingHoles, U1 MAX3232

Commit message: Updated Design v1.0
Parts:
- added REF**: MountingHole_3.2mm_M3_ISO14580_Pad, MountingHole:MountingHole_3.2mm_M3_ISO14580_Pad, F.Cu at (88.1, 94.4)
- added REF**: MountingHole_3.2mm_M3_ISO14580_Pad, MountingHole:MountingHole_3.2mm_M3_ISO14580_Pad, F.Cu at (30.1, 94.4)
- added REF**: MountingHole_3.2mm_M3_ISO14580_Pad, MountingHole:MountingHole_3.2mm_M3_ISO14580_Pad, F.Cu at (30.1, 71.4)
- added REF**: MountingHole_3.2mm_M3_ISO14580_Pad, MountingHole:MountingHole_3.2mm_M3_ISO14580_Pad, F.Cu at (88.1, 71.5)
Other:
- outline, holes or cut-outs redrawn
Changed lines of the file:
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@@
   (general
     (thickness 1.6)
-    (drawings 1028)
+    (drawings 1024)
     (tracks 152)
     (zones 0)
-    (modules 10)
+    (modules 14)
     (nets 13)
   )
@@
     (solder_mask_min_width 0.25)
     (aux_axis_origin 0 0)
+    (grid_origin 91.7702 67.9196)
     (visible_elements FFFFFF7F)
     (pcbplotparams
@@
     (add_net "Net-(C3-Pad2)")
     (add_net "Net-(C4-Pad1)")
+  )
+  (module MountingHole:MountingHole_3.2mm_M3_ISO14580_Pad (layer F.Cu)
+    (at 88.138 94.4372)
+    (descr "Mounting Hole 3.2mm, M3, ISO14580")
+    (tags "mounting hole 3.2mm m3 iso14580")
+    (attr virtual)
+    (fp_text reference REF** (at 0 -3.75) (layer F.SilkS) hide
+      (effects (font (size 1 1) (thickness 0.15)))
+    )
+    (fp_text value MountingHole_3.2mm_M3_ISO14580_Pad (at 0 3.75) (layer F.Fab) hide
+      (effects (font (size 1 1) (thickness 0.15)))
+    )
+    (fp_text user %R (at 0.3 0) (layer F.Fab) hide
+      (effects (font (size 1 1) (thickness 0.15)))
+    )
+    (fp_circle (center 0 0) (end 2.75 0) (layer Cmts.User) (width 0.15))
+    (fp_circle (center 0 0) (end 3 0) (layer F.CrtYd) (width 0.05))
+    (pad 1 thru_hole circle (at 0 0) (size 5.5 5.5) (drill 3.2) (layers *.Cu *.Mask))
+  )
+  (module MountingHole:MountingHole_3.2mm_M3_ISO14580_Pad (layer F.Cu)
+    (at 30.099 94.4372)
+    (descr "Mounting Hole 3.2mm, M3, ISO14580")
+    (tags "mounting hole 3.2mm m3 iso14580")
+    (attr virtual)
+    (fp_text reference REF** (at 0 -3.75) (layer F.SilkS) hide
+      (effects (font (size 1 1) (thickness 0.15)))
+    )
+    (fp_text value MountingHole_3.2mm_M3_ISO14580_Pad (at 0 3.75) (layer F.Fab) hide
+      (effects (font (size 1 1) (thickness 0.15)))
+    )
+    (fp_text user %R (at 0.3 0) (layer F.Fab) hide
+      (effects (font (size 1 1) (thickness 0.15)))
+    )
+    (fp_circle (center 0 0) (end 2.75 0) (layer Cmts.User) (width 0.15))
+    (fp_circle (center 0 0) (end 3 0) (layer F.CrtYd) (width 0.05))
+    (pad 1 thru_hole circle (at 0 0) (size 5.5 5.5) (drill 3.2) (layers *.Cu *.Mask))
+  )
+  (module MountingHole:MountingHole_3.2mm_M3_ISO14580_Pad (layer F.Cu)
+    (at 30.099 71.4248)
+    (descr "Mounting Hole 3.2mm, M3, ISO14580")
+    (tags "mounting hole 3.2mm m3 iso14580")
+    (attr virtual)
+    (fp_text reference REF** (at 0 -3.75) (layer F.SilkS) hide
+      (effects (font (size 1 1) (thickness 0.15)))
+    )
+    (fp_text value MountingHole_3.2mm_M3_ISO14580_Pad (at 0 3.75) (layer F.Fab) hide
+      (effects (font (size 1 1) (thickness 0.15)))
+    )
+    (fp_text user %R (at 0.3 0) (layer F.Fab) hide
+      (effects (font (size 1 1) (thickness 0.15)))
+    )
+    (fp_circle (center 0 0) (end 2.75 0) (layer Cmts.User) (width 0.15))
+    (fp_circle (center 0 0) (end 3 0) (layer F.CrtYd) (width 0.05))
+    (pad 1 thru_hole circle (at 0 0) (size 5.5 5.5) (drill 3.2) (layers *.Cu *.Mask))
+  )
+  (module MountingHole:MountingHole_3.2mm_M3_ISO14580_Pad (layer F.Cu)
+    (at 88.138 71.4502)
+    (descr "Mounting Hole 3.2mm, M3, ISO14580")
+    (tags "mounting hole 3.2mm m3 iso14580")
+    (attr virtual)
+    (fp_text reference REF** (at 0 -3.75) (layer F.SilkS) hide
+      (effects (font (size 1 1) (thickness 0.15)))
+    )
+    (fp_text value MountingHole_3.2mm_M3_ISO14580_Pad (at 0 3.75) (layer F.Fab) hide
+      (effects (font (size 1 1) (thickness 0.15)))
+    )
+    (fp_circle (center 0 0) (end 3 0) (layer F.CrtYd) (width 0.05))
+    (fp_circle (center 0 0) (end 2.75 0) (layer Cmts.User) (width 0.15))
+    (fp_text user %R (at 0.3 0) (layer F.Fab) hide
+      (effects (font (size 1 1) (thickness 0.15)))
+    )
+    (pad 1 thru_hole circle (at 0 0) (size 5.5 5.5) (drill 3.2) (layers *.Cu *.Mask))
   )
   (module Symbol:OSHW-Logo2_14.6x12mm_SilkScreen (layer B.Cu)
@@
     )
   )
+  (gr_line (start 91.7702 67.9196) (end 85.8774 67.9196) (layer Edge.Cuts) (width 0.05))
   (gr_text "Concept by Mr Lurch\nDesign by dJOS" (at 60.0456 82.2706) (layer B.SilkS)
     (effects (font (size 1 1) (thickness 0.2)) (justify mirror))
@@
     (effects (font (size 2 2) (thickness 0.3)) (justify mirror))
   )
-  (gr_circle (center 30.099 71.4248) (end 31.8262 71.6534) (layer Edge.Cuts) (width 0.05))
-  (gr_circle (center 30.099 94.4372) (end 31.8262 94.6658) (layer Edge.Cuts) (width 0.05))
-  (gr_circle (center 88.138 94.4626) (end 89.8652 94.6912) (layer Edge.Cuts) (width 0.05))
-  (gr_line (start 91.7702 67.9196) (end 85.8774 67.9196) (layer Edge.Cuts) (width 0.05))
   (gr_line (start 26.5684 67.8942) (end 26.6192 97.9424) (layer Edge.Cuts) (width 0.05))
-  (gr_circle (center 88.138 71.4756) (end 89.8652 71.7042) (layer Edge.Cuts) (width 0.05))
   (gr_line (start 91.7702 67.9196) (end 91.7956 97.9424) (layer Edge.Cuts) (width 0.1))
   (gr_line (start 85.8774 55.9308) (end 85.8774 67.9196) (layer Edge.Cuts) (width 0.1))
